Commit message: start integration of the robot_movement_config-pkg

File: launch/volksbot_r6.urdf (robot description, URDF)
Before this commit: robot volksbot_r6, 10 links, 9 joints
Links:
- link left_tread: geometry visual cylinder length=0.06 radius=0.108
- link right_tread: geometry visual cylinder length=0.06 radius=0.108

Commit message: working config with prototype of robot_movement_config

File: launch/volksbot_r6.urdf (robot description, URDF)
Before this commit: robot volksbot_r6, 10 links, 9 joints
Joints:
- removed joint wheels_left
- removed joint wheels_left_2
- removed joint wheels_right
- removed joint wheels_right_2
- added joint left_tread: type continuous, parent left_tread, child wheel_front_left, origin xyz=0.23 0 0 rpy=0 0 0, axis 0 0 1
- added joint left_tread_2: type continuous, parent left_tread, child wheel_rear_left, origin xyz=-0.23 0 0 rpy=0 0 0, axis 0 0 1, mimic joint=left_tread
- added joint right_tread: type continuous, parent right_tread, child wheel_front_right, origin xyz=0.23 0 0 rpy=0 0 0, axis 0 0 1
- added joint right_tread_2: type continuous, parent right_tread, child wheel_rear_right, origin xyz=-0.23 0 0 rpy=0 0 0, axis 0 0 1, mimic joint=right_tread
